File: Production/14044-sparkfun-mlx90640-qwiic-breakout-Panel.brd (EAGLE design)
At the start: 226.8 x 149.1 mm, 1443 parts, among them J101 PTH, J104 PTH, J107 PTH, J11 PTH, J110 PTH, J113 PTH, J116 PTH, J119 PTH, J14 PTH, J17 PTH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

Commit message: panel
Parts:
- removed E$1, E$2: (no value), SparkFun-Aesthetics:FIDUCIAL-1X2
- added E$7, E$8: (no value), SparkFun-Aesthetics:FIDUCIAL-1X2
- moved E$3 11.1 mm to (-3.05, 2.98)
Other:
- board size 226.8 x 149.1 mm -> 220.5 x 142.7 mm
- board text added: "v11"
- board text removed: "v-score"
- board text removed: "v10"
